File: src/elec/lightbarriersync/lightbarriersync.kicad_pcb (KiCad board)
At the start: 2 copper layers, 20.1 x 40.5 mm, 52 parts, among them J1 Conn_01x03_Pin, Q1 MMBFJ113, Q10 BC850, Q11 2N7002, Q12 2N7002, Q2 2N7002, Q3 2N7002, Q4 BC850, Q5 BC850, Q6 BC850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

Commit message: board ready
Parts:
- added REF**: KiCad-Logo2_5mm_SilkScreen, Symbol:KiCad-Logo2_5mm_SilkScreen, B.Cu at (50.2, 27.5)
- moved R6 0.16 mm to (40.6, 17.9)
- moved D1 0.13 mm to (41.4, 15.1)
Routing:
- net GND: track 30.8 -> 31.5 mm, vias 11 -> 10
- added copper zone on B.Cu, net GND
- added copper zone on F.Cu, net GND
Other:
- board size 20.1 x 40.5 mm -> 20.3 x 40.5 mm
- board text added: "${VERSION}"
- board text added: "https://github.com/TheTesla/lightbarriersync"
- board text added: "recv"
- board text added: "send"
