File: src/elec/lightbarriersync/lightbarriersync.kicad_sch (KiCad schematic)
At the start: 50 parts, among them J1 Conn_01x03_Pin, Q1 MMBFJ113, Q10 BC850, Q11 2N7002, Q12 2N7002, Q2 2N7002, Q3 2N7002, Q4 BC850, Q5 BC850, Q6 BC850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

Commit message: board ready
Other:
- company: (none) -> ${ORG}
- title: (none) -> ${TITLE}
Changed lines of the file:
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@@
 	(generator_version "9.0")
 	(paper "A4")
+	(title_block
+		(title "${TITLE}")
+		(date "2026-04-18")
+		(rev "${VERSION}")
+		(company "${ORG}")
+		(comment 1 "${NAME}")
+	)
 	(junction
 		(at 74.93 72.39)
