File: src/elec/lightbarriersyncopamp/lightbarriersyncopamp.kicad_pcb (KiCad board)
At the start: 2 copper layers, 18.2 x 45 mm, 46 parts, among them J1 Conn_01x03_Pin, Q1 BSS84, Q2 BSS123, Q3 BC850, Q4 BSS123, Q5 BSS123, Q6 BC850, Q7 BSS123, U1 LP2951-3.3_SOIC, U2 LM324A

Commit message: addec copyright; ToDo: variables, version, opamp variant note, data on silkscreen
Parts:
- added REF**: OSHW-Logo2_14.6x12mm_SilkScreen, Symbol:OSHW-Logo2_14.6x12mm_SilkScreen, B.Cu at (111.5, 100.7)
Other:
- board text added: "Copyright (c) 2026 Stefan Helmert <stefan@entroserv.de>"
- board text added: "https://github.com/TheTesla/lightbarriersync"

Commit message: ready to build
Parts:
- removed the REF** at (111.5, 100.7)
- added C7: 2u2, Capacitor_SMD:C_0805_2012Metric, F.Cu at (111.6, 126.3)
- added REF**: KiCad-Logo2_5mm_SilkScreen, Symbol:KiCad-Logo2_5mm_SilkScreen, B.Cu at (111.7, 100.3)
- added REF**: OSHW-Logo2_7.3x6mm_SilkScreen, Symbol:OSHW-Logo2_7.3x6mm_SilkScreen, B.Cu at (114.5, 88.8)
- R1: value 12k -> 10k
- U2: value LM324A -> TLV9004IDR
Routing:
- net VIN: track 33.5 -> 36.7 mm, vias 0 -> 1
- net Net-(D5-A): track 16.4 -> 18.6 mm, vias 0 -> 2
- net Net-(D8-A): track 4.06 -> 6.09 mm
Other:
- board text added: "${TITLE} ${VERSION}"
- board text added: "Us:3..30V Is<2mA fir~70kHz Iosnk<0.5mA Uosnk~0.4V"
