File: src/elec/lightbarriersyncopamp/lightbarriersyncopamp.kicad_sch (KiCad schematic)
At the start: 46 parts, among them J1 Conn_01x03_Pin, Q1 BSS84, Q2 BSS123, Q3 BC850, Q4 BSS123, Q5 BSS123, Q6 BC850, Q7 BSS123, U1 LP2951-3.3_SOIC, U2 LM324A

Commit message: restored
Parts:
- U2: value LM324A -> TLV9004IDR
Changed lines of the file:
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@@
 			)
 		)
-		(property "Value" "LM324A"
+		(property "Value" "TLV9004IDR"
 			(at 119.38 180.3399 0)
 			(show_name no)
@@
 			)
 		)
-		(property "Datasheet" "http://www.ti.com/lit/ds/symlink/lm2902-n.pdf"
+		(property "Datasheet" "https://www.ti.com/lit/ds/symlink/tlv9004.pdf"
 			(at 121.92 173.99 0)
 			(hide yes)
@@
 			)
 		)
-		(property "Description" "Low-Power, Quad-Operational Amplifiers, DIP-14/SOIC-14/SSOP-14"
+		(property "Description" "Low-Power RRIO Quad-Operational Amplifiers, SOIC-14"
 			(at 120.65 179.07 0)
 			(hide yes)
@@
 			)
 		)
-		(property "Value" "LM324A"
+		(property "Value" "TLV9004IDR"
 			(at 78.74 55.88 0)
 			(show_name no)
@@
 			)
 		)
-		(property "Datasheet" "http://www.ti.com/lit/ds/symlink/lm2902-n.pdf"
+		(property "Datasheet" "https://www.ti.com/lit/ds/symlink/tlv9004.pdf"
 			(at 80.01 58.42 0)
 			(hide yes)
@@
 			)
 		)
-		(property "Description" "Low-Power, Quad-Operational Amplifiers, DIP-14/SOIC-14/SSOP-14"
+		(property "Description" "Low-Power RRIO Quad-Operational Amplifiers, SOIC-14"
 			(at 78.74 63.5 0)
 			(hide yes)
@@
 			)
 		)
-		(property "Value" "LM324A"
+		(property "Value" "TLV9004IDR"
 			(at 64.77 119.38 0)
 			(show_name no)
@@
 			)
 		)
-		(property "Datasheet" "http://www.ti.com/lit/ds/symlink/lm2902-n.pdf"
+		(property "Datasheet" "https://www.ti.com/lit/ds/symlink/tlv9004.pdf"
 			(at 66.04 121.92 0)
 			(hide yes)
@@
 			)
 		)
-		(property "Description" "Low-Power, Quad-Operational Amplifiers, DIP-14/SOIC-14/SSOP-14"
+		(property "Description" "Low-Power RRIO Quad-Operational Amplifiers, SOIC-14"
 			(at 64.77 127 0)
 			(hide yes)
@@
 			)
 		)
-		(property "Value" "LM324A"
+		(property "Value" "TLV9004IDR"
 			(at 53.34 55.88 0)
 			(show_name no)
@@
 			)
 		)
-		(property "Datasheet" "http://www.ti.com/lit/ds/symlink/lm2902-n.pdf"
+		(property "Datasheet" "https://www.ti.com/lit/ds/symlink/tlv9004.pdf"
 			(at 54.61 58.42 0)
 			(hide yes)
@@
 			)
 		)
-		(property "Description" "Low-Power, Quad-Operational Amplifiers, DIP-14/SOIC-14/SSOP-14"
+		(property "Description" "Low-Power RRIO Quad-Operational Amplifiers, SOIC-14"
 			(at 53.34 63.5 0)
 			(hide yes)
@@
 			)
 		)
-		(property "Value" "LM324A"
+		(property "Value" "TLV9004IDR"
 			(at 130.81 119.38 0)
 			(show_name no)
@@
 			)
 		)
-		(property "Datasheet" "http://www.ti.com/lit/ds/symlink/lm2902-n.pdf"
+		(property "Datasheet" "https://www.ti.com/lit/ds/symlink/tlv9004.pdf"
 			(at 132.08 121.92 0)
 			(hide yes)
@@
 			)
 		)
-		(property "Description" "Low-Power, Quad-Operational Amplifiers, DIP-14/SOIC-14/SSOP-14"
+		(property "Description" "Low-Power RRIO Quad-Operational Amplifiers, SOIC-14"
 			(at 130.81 127 0)
 			(hide yes)

Commit message: ready to build
Parts:
- added C7: 2u2, Capacitor_SMD:C_0805_2012Metric, symbol Device:C_Small
- D3: value LD271 -> WP7113F3BT
- D6: value SFH203 -> WP7113PD1BT
- R1: value 12k -> 10k
Connections:
- net GND: now also C7.2
- net VIN: now also C7.1
- no-connect marks 0 -> 3
Other:
- company: Stefan Helmert -> ${ORG}
- title: Lightbarrier Snyc Op -> ${TITLE}
- moved on the sheet: D4
Changed lines of the file:
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@@
 	(paper "A4")
 	(title_block
-		(title "Lightbarrier Snyc Op")
+		(title "${TITLE}")
 		(date "2026-05-15")
-		(rev "0.1")
-		(company "Stefan Helmert")
-		(comment 1 "entroserv.de")
+		(rev "${VERSION}")
+		(company "${ORG}")
+		(comment 1 "${NAME}")
 	)
 	(junction
@@
 	)
 	(junction
+		(at 52.07 190.5)
+		(diameter 0)
+		(color 0 0 0 0)
+	)
+	(junction
 		(at 38.1 60.96)
 		(diameter 0)
@@
 	)
 	(junction
+		(at 39.37 168.91)
+		(diameter 0)
+		(color 0 0 0 0)
+	)
+	(junction
 		(at 149.86 127)
 		(diameter 0)
@@
 		(color 0 0 0 0)
 	)
+	(no_connect
+		(at 91.44 181.61)
+	)
+	(no_connect
+		(at 91.44 176.53)
+	)
+	(no_connect
+		(at 91.44 171.45)
+	)
 	(wire
 		(pts
@@
 	(wire
 		(pts
+			(xy 52.07 190.5) (xy 39.37 190.5)
+		)
+		(stroke
+			(width 0)
+			(type default)
+		)
+	)
+	(wire
+		(pts
 			(xy 45.72 66.04) (xy 43.18 66.04)
 		)
@@
 	(wire
 		(pts
+			(xy 39.37 190.5) (xy 39.37 186.69)
+		)
+		(stroke
+			(width 0)
+			(type default)
+		)
+	)
+	(wire
+		(pts
 			(xy 44.45 129.54) (xy 44.45 133.35)
 		)
@@
 	(wire
 		(pts
+			(xy 39.37 181.61) (xy 39.37 168.91)
+		)
+		(stroke
+			(width 0)
+			(type default)
+		)
+	)
+	(wire
+		(pts
 			(xy 101.6 87.63) (xy 101.6 85.09)
 		)
@@
 			)
 		)
-		(property "Value" "SFH203"
+		(property "Value" "WP7113PD1BT"
 			(at 29.21 142.5828 90)
 			(show_name no)
@@
 			)
 		)
-		(property "Datasheet" "http://www.osram-os.com/Graphics/XPic9/00101656_0.pdf/SFH%20203,%20SFH%20203%20FA,%20Lead%20(Pb)%20Free%20Product%20-%20RoHS%20Compliant.pdf"
+		(property "Datasheet" "https://www.kingbrightusa.com/images/catalog/SPEC/WP7113PD1BT-BD-P22.pdf"
 			(at 24.13 140.97 0)
 			(hide yes)
@@
 	)
 	(symbol
+		(lib_id "Device:C_Small")
+		(at 39.37 184.15 0)
+		(unit 1)
+		(body_style 1)
+		(exclude_from_sim no)
+		(in_bom yes)
+		(on_board yes)
+		(in_pos_files yes)
+		(dnp no)
+		(fields_autoplaced yes)
+		(property "Reference" "C7"
+			(at 41.91 182.8862 0)
+			(show_name no)
+			(do_not_autoplace no)
+			(effects
+				(font
+					(size 1.27 1.27)
+				)
+				(justify left)
+			)
+		)
+		(property "Value" "2u2"
+			(at 41.91 185.4262 0)
+			(show_name no)
+			(do_not_autoplace no)
+			(effects
+				(font
+					(size 1.27 1.27)
+				)
+				(justify left)
+			)
+		)
+		(property "Footprint" "Capacitor_SMD:C_0805_2012Metric"
+			(at 39.37 184.15 0)
+			(hide yes)
+			(show_name no)
+			(do_not_autoplace no)
+			(effects
+				(font
+					(size 1.27 1.27)
+				)
+			)
+		)
+		(property "Datasheet" ""
+			(at 39.37 184.15 0)
+			(hide yes)
+			(show_name no)
+			(do_not_autoplace no)
+			(effects
+				(font
+					(size 1.27 1.27)
+				)
+			)
+		)
+		(property "Description" "Unpolarized capacitor, small symbol"
+			(at 39.37 184.15 0)
+			(hide yes)
+			(show_name no)
+			(do_not_autoplace no)
+			(effects
+				(font
+					(size 1.27 1.27)
+				)
+			)
+		)
+		(pin "1"
+		)
+		(pin "2"
+		)
+		(instances
+			(project "lightbarriersyncopamp"
+				(path "/25642f40-c577-4c48-9e64-fb6733cf316e"
+					(reference "C7")
+					(unit 1)
+				)
+			)
+		)
+	)
+	(symbol
 		(lib_id "Device:R_Small")
 		(at 161.29 138.43 0)
@@
 			)
 		)
-		(property "Value" "LD271"
+		(property "Value" "WP7113F3BT"
 			(at 115.57 46.8629 90)
 			(show_name no)
@@
 			)
 		)
-		(property "Datasheet" "http://www.alliedelec.com/m/d/40788c34903a719969df15f1fbea1056.pdf"
+		(property "Datasheet" "https://www.kingbrightusa.com/images/catalog/SPEC/WP7113F3BT.pdf"
 			(at 113.03 45.72 0)
 			(hide yes)
@@
 	(symbol
 		(lib_id "Diode:1N4148W")
-		(at 54.61 140.97 90)
+		(at 54.61 140.97 270)
+		(mirror x)
 		(unit 1)
 		(body_style 1)
@@
 		(in_pos_files yes)
 		(dnp no)
-		(fields_autoplaced yes)
 		(property "Reference" "D4"
-			(at 57.15 139.6999 90)
+			(at 52.07 139.6999 90)
 			(show_name no)
 			(do_not_autoplace no)
@@
 		)
 		(property "Value" "1N4148W"
-			(at 57.15 142.2399 90)
+			(at 52.07 142.2399 90)
 			(show_name no)
 			(do_not_autoplace no)
@@
 		)
 		(property "Footprint" "Diode_SMD:D_SOD-123"
-			(at 59.055 140.97 0)
+			(at 50.165 140.97 0)
 			(hide yes)
 			(show_name no)
@@
 			)
 		)
-		(property "Value" "12k"
+		(property "Value" "10k"
 			(at 104.14 187.96 0)
 			(show_name no)

Commit message: version 0.2 optimized with less components
Parts:
- removed D4: 1N4148W, Diode_SMD:D_SOD-123, symbol Diode:1N4148W
- removed R10, R15, R9: 10k, Resistor_SMD:R_0805_2012Metric, symbol Device:R_Small
- C5: value 100n -> 1n
Connections:
- net at U2.10 (+): now also D7.2 (A), R18.2, R19.1, U2.5 (+)
Other:
- moved on the sheet: C1, C2, C3, C4, C5, C6, C7, D1, D2, D3, D5, D6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
